Commit message: added hardware dual arm control

File: assets/universal_robots_ur5e/dual_ur5e.urdf (robot description, URDF)
Before this commit: robot dual_ur5e_robot, 23 links, 22 joints
Joints:
- joint world_to_left_arm_base: origin xyz=0 0.275 0.3 rpy=0 -0.7853981633974483 -1.5707963267948966 -> xyz=0 0.275 0.3 rpy=0.7853981633974483 0 3.141592653589793
- joint world_to_right_arm_base: origin xyz=0 -0.275 0.3 rpy=0 -0.7853981633974483 1.5707963267948966 -> xyz=0 -0.275 0.3 rpy=0.7853981633974483 0 0
