Commit message: added dual galaxea a1x arm mujoco demo

File: assets/galaxea/A1X/a1x.urdf (robot description, URDF)
Before this commit: robot A1X, 10 links, 9 joints
Links:
- link arm_link1: geometry collision mesh filename=meshes/arm_link1.STL; visual mesh filename=meshes/arm_link1.STL
- link arm_link2: geometry collision mesh filename=meshes/arm_link2.STL; visual mesh filename=meshes/arm_link2.STL
- link arm_link3: geometry collision mesh filename=meshes/arm_link3.STL; visual mesh filename=meshes/arm_link3.STL
- link arm_link4: geometry collision mesh filename=meshes/arm_link4.STL; visual mesh filename=meshes/arm_link4.STL
- link arm_link5: geometry collision mesh filename=meshes/arm_link5.STL; visual mesh filename=meshes/arm_link5.STL
- link arm_link6: geometry collision mesh filename=meshes/arm_link6.STL; visual mesh filename=meshes/arm_link6.STL
- link base_link: geometry collision mesh filename=meshes/base_link.STL; visual mesh filename=meshes/base_link.STL
- link gripper_finger_link1: geometry collision mesh filename=meshes/gripper_finger_link1.STL; visual mesh filename=meshes/gripper_finger_link1.STL
- link gripper_finger_link2: geometry collision mesh filename=meshes/gripper_finger_link2.STL; visual mesh filename=meshes/gripper_finger_link2.STL
- link gripper_link: geometry collision mesh filename=meshes/gripper_link.STL; visual mesh filename=meshes/gripper_link.STL
